Commit message: Changed the URDF according to Rviz. Physics might be wonky

File: src/cypher_description/urdf/cypher_body.urdf (robot description, URDF)
Before this commit: robot rocker_bogie_bot_fixed, 12 links, 11 joints
Links:
- link base_link: geometry collision box size=0.49 0.35 0.1874; visual box size=0.49 0.35 0.1874
- link left_bogie: geometry collision box size=0.25 0.06 0.04; visual box size=0.25 0.06 0.04
- link left_front_wheel: geometry collision cylinder length=0.04 radius=0.075; visual cylinder length=0.04 radius=0.075
- link left_middle_wheel: geometry collision cylinder length=0.04 radius=0.075; visual cylinder length=0.04 radius=0.075
- link left_rear_wheel: geometry collision cylinder length=0.04 radius=0.075; visual cylinder length=0.04 radius=0.075
- link left_rocker: geometry collision box size=0.2 0.06 0.04; visual box size=0.2 0.06 0.04
- link right_bogie: geometry collision box size=0.25 0.06 0.04; visual box size=0.25 0.06 0.04
- link right_front_wheel: geometry collision cylinder length=0.04 radius=0.075; visual cylinder length=0.04 radius=0.075
- link right_middle_wheel: geometry collision cylinder length=0.04 radius=0.075; visual cylinder length=0.04 radius=0.075
- link right_rear_wheel: geometry collision cylinder length=0.04 radius=0.075; visual cylinder length=0.04 radius=0.075
- link right_rocker: geometry collision box size=0.2 0.06 0.04; visual box size=0.2 0.06 0.04

Commit message: URDF Changed. no Physics yet

File: src/cypher_description/urdf/cypher_body.urdf (robot description, URDF)
Before this commit: robot rocker_bogie_bot_fixed, 12 links, 11 joints
Links:
- removed link imu_link
- removed link left_bogie
- removed link left_middle_wheel
- removed link left_rocker
- removed link right_bogie
- removed link right_middle_wheel
- removed link right_rocker
- added link left_bogie_horizontal_strip; visual box size=0.38 0.025 0.003
- added link left_bogie_rear_wheel_strip; visual box size=0.183 0.025 0.003
- added link left_bogie_to_rocker_strip; visual box size=0.043 0.025 0.003
- added link left_mid_wheel; visual cylinder length=0.04 radius=0.075
- added link left_rocker_frontwheel_strip; visual box size=0.161 0.025 0.003
- added link left_rocker_midwheel_strip; visual box size=0.147 0.025 0.003
- added link right_bogie_horizontal_strip; visual box size=0.38 0.025 0.003
- added link right_bogie_rear_wheel_strip; visual box size=0.183 0.025 0.003
- added link right_bogie_to_rocker_strip; visual box size=0.043 0.025 0.003
- added link right_mid_wheel; visual cylinder length=0.04 radius=0.075
- added link right_rocker_frontwheel_strip; visual box size=0.161 0.025 0.003
- added link right_rocker_midwheel_strip; visual box size=0.147 0.025 0.003
- link base_link: mass 6.0 -> None; geometry visual box size=0.49 0.35 0.02
- link left_front_wheel: mass 0.3 -> None; geometry visual cylinder length=0.04 radius=0.075
- link left_rear_wheel: mass 0.3 -> None; geometry visual cylinder length=0.04 radius=0.075
- link right_front_wheel: mass 0.3 -> None; geometry visual cylinder length=0.04 radius=0.075
- link right_rear_wheel: mass 0.3 -> None; geometry visual cylinder length=0.04 radius=0.075
Joints:
- removed joint imu_joint
- removed joint left_bogie_joint
- removed joint left_middle_wheel_joint
- removed joint left_rear_wheel_joint
- removed joint right_bogie_joint
- removed joint right_middle_wheel_joint
- removed joint right_rear_wheel_joint
- added joint left_Bogie_to_Base_chassis_joint: type revolute, parent base_link, child left_bogie_horizontal_strip, origin xyz=0.245 -0.175 0.2233 rpy=0 0 0, axis 0 1 0, limit lower=-1.5708 upper=1.5708 effort=50 velocity=1.0
- added joint left_bogie_to_rocker_joint: type fixed, parent left_bogie_horizontal_strip, child left_bogie_to_rocker_strip, origin xyz= -0.195 -0.175 0.15 rpy=0 0 0, axis 0 0 0
- added joint left_front_mid_joint: type continuous, parent left_rocker_midwheel_strip, child left_mid_wheel, origin xyz= -0.1 -0.175 0.075 rpy=0 0 0, axis 0 1 0
- added joint left_front_rear_joint: type continuous, parent left_bogie_rear_wheel_strip, child left_rear_wheel, origin xyz= 0.25 -0.175 0.075 rpy=0 0 0, axis 0 1 0
- added joint left_rear_wheel_strip_to_horizontal_strip: type fixed, parent left_bogie_horizontal_strip, child left_bogie_rear_wheel_strip, origin xyz=0.195 -0.175 0.2233 rpy=0 0 0, axis 0 0 0
- added joint left_rocker_joint_to_bogie: type revolute, parent left_bogie_horizontal_strip, child left_rocker_frontwheel_strip, origin xyz= -0.195 -0.175 0.138 rpy=0 0 0, axis 0 0 0, limit lower=-1.5708 upper=1.5708 effort=50 velocity=1.0
- added joint rear_wheel_strip_to_horizontal_strip: type fixed, parent right_bogie_horizontal_strip, child right_bogie_rear_wheel_strip, origin xyz=0.195 0.175 0.2233 rpy=0 0 0, axis 0 0 0
- added joint right_Bogie_to_Base_chassis_joint: type revolute, parent base_link, child right_bogie_horizontal_strip, origin xyz=0.245 0.175 0.2233 rpy=0 0 0, axis 0 1 0, limit lower=-1.5708 upper=1.5708 effort=50 velocity=1.0
- added joint right_bogie_to_rocker_joint: type fixed, parent right_bogie_horizontal_strip, child right_bogie_to_rocker_strip, origin xyz= -0.195 0.175 0.15 rpy=0 0 0, axis 0 0 0
- added joint right_front_mid_joint: type continuous, parent right_rocker_midwheel_strip, child right_mid_wheel, origin xyz= -0.1 0.175 0.075 rpy=0 0 0, axis 0 1 0
- added joint right_front_rear_joint: type continuous, parent right_bogie_rear_wheel_strip, child right_rear_wheel, origin xyz= 0.25 0.175 0.075 rpy=0 0 0, axis 0 1 0
- added joint right_rocker_joint_to_bogie: type revolute, parent right_bogie_horizontal_strip, child right_rocker_frontwheel_strip, origin xyz= -0.195 0.175 0.138 rpy=0 0 0, axis 0 0 0, limit lower=-1.5708 upper=1.5708 effort=50 velocity=1.0
- joint left_front_wheel_joint: origin xyz=0.16117 0 -0.075 rpy=0 0 0 -> xyz= -0.3 -0.175 0.075 rpy=0 0 0; parent left_rocker -> left_rocker_frontwheel_strip
- joint left_rocker_joint: axis 0 1 0 -> 0 0 0; child left_rocker -> left_rocker_midwheel_strip; limit lower=-1.5708 upper=1.5708 effort=50 velocity=1.0 -> (none); origin xyz=0 0.175 0 rpy=0 0 0 -> xyz= -0.195 -0.175 0.138 rpy=0 0 0; parent base_link -> left_rocker_frontwheel_strip; type revolute -> fixed
- joint right_front_wheel_joint: origin xyz=0.16117 0 -0.075 rpy=0 0 0 -> xyz= -0.3 0.175 0.075 rpy=0 0 0; parent right_rocker -> right_rocker_frontwheel_strip
- joint right_rocker_joint: axis 0 1 0 -> 0 0 0; child right_rocker -> right_rocker_midwheel_strip; limit lower=-1.5708 upper=1.5708 effort=50 velocity=1.0 -> (none); origin xyz=0 -0.175 0 rpy=0 0 0 -> xyz= -0.195 0.175 0.138 rpy=0 0 0; parent base_link -> right_rocker_frontwheel_strip; type revolute -> fixed
